File: hardware/eagle/Inputs/Input-Model1.brd (EAGLE design)
At the start: 32.7 x 82.5 mm, 34 parts

Commit message: Module configuration
Parts:
- moved R16 1.03 mm to (23.9, 4.81), flipped to the bottom
- moved R10 0.26 mm to (23.9, 62.2), flipped to the bottom
- moved R11 0.26 mm to (23.9, 52.1), flipped to the bottom
- moved R12 0.26 mm to (23.9, 41.9), flipped to the bottom
- moved R13 0.26 mm to (23.9, 31.8), flipped to the bottom
- moved R14 0.26 mm to (23.9, 21.6), flipped to the bottom
- moved R15 0.26 mm to (23.9, 11.4), flipped to the bottom
- moved R9 0.26 mm to (23.9, 72.4), flipped to the bottom
- moved R1 0.06 mm to (14.0, 78.7), flipped to the bottom
- moved R2 0.06 mm to (14.0, 68.6), flipped to the bottom
- moved R3 0.06 mm to (14.0, 58.4), flipped to the bottom
- moved R4 0.06 mm to (14.0, 48.3), flipped to the bottom
- moved R5 0.06 mm to (14.0, 38.1), flipped to the bottom
- moved R6 0.06 mm to (14.0, 27.9), flipped to the bottom
- moved R7 0.06 mm to (14.0, 17.8), flipped to the bottom
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Routing:
- net N$2: track 200.8 -> 195.4 mm
- net N$10: track 30.4 -> 28.9 mm
Other:
- board size 32.7 x 82.5 mm -> 34.7 x 85.5 mm

Commit message: Melhorias nos processos de comunicação com o Arduino
Parts:
- moved R10 11.0 mm to (34.9, 63.2)
- moved R11 11.0 mm to (34.9, 53.1)
- moved R12 11.0 mm to (34.9, 42.9)
- moved R13 11.0 mm to (34.9, 32.8)
- moved R14 11.0 mm to (34.9, 22.6)
- moved R15 11.0 mm to (34.9, 12.4)
- moved R9 11.0 mm to (34.9, 73.4)
- moved R1 11.0 mm to (3.03, 78.7)
- moved R2 11.0 mm to (3.03, 68.6)
- moved R3 11.0 mm to (3.03, 58.4)
- moved R4 11.0 mm to (3.03, 48.3)
- moved R5 11.0 mm to (3.03, 38.1)
- moved R6 11.0 mm to (3.03, 27.9)
- moved R7 11.0 mm to (3.03, 17.8)
- moved R8 11.0 mm to (3.03, 7.62)
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Routing:
- net N$2: track 195.4 -> 345.5 mm
- net N$3: track 194.1 -> 268.4 mm
- net N$9: track 31.6 -> 4.72 mm
- net N$5: track 12.5 -> 17.2 mm
- net N$15: track 12.5 -> 17.1 mm
- net N$6: track 14.4 -> 18.3 mm
- net N$11: track 45.1 -> 42.5 mm
- net N$16: track 16.0 -> 18.2 mm
- net N$12: track 37.5 -> 35.3 mm
- net N$14: track 18.2 -> 20.3 mm
- net N$8: track 39.2 -> 37.4 mm
- net N$1: track 29.0 -> 27.2 mm
- net N$13: track 26.0 -> 27.8 mm
- net N$17: track 23.6 -> 22.0 mm
- net N$4: track 19.2 -> 20.4 mm
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Other:
- board size 34.7 x 85.5 mm -> 38.7 x 85.5 mm
